File: ColoLightCustom.kicad_sch (KiCad schematic)
At the start: 4 parts, among them J1 Conn_01x05_Male, J2 Conn_01x05_Male, J3 Conn_01x03, J4 Conn_01x03_Male

Commit message: v0.3
Parts:
- J3: footprint halibs:SolderPads3 -> haus-automatisierung:SolderPads3
Changed lines of the file:
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@@
 			)
 		)
-		(property "Footprint" "halibs:SolderPads3"
+		(property "Footprint" "haus-automatisierung:SolderPads3"
 			(at 186.69 93.98 0)
 			(effects
